Commit message: Updated for realsense and depth sensor integration for rov_localization. May not work in sim now <- updates needed

File: urdf/rov_base.xacro (robot description, xacro)
@@ -17,11 +17,11 @@
     <!-- base_link according to ROS conventions: x forward, z up -->
     <link name="${namespace}/base_link">
-      <inertial>
-        <mass value="${mass}"/>
-        <origin xyz="0.00056715 0.0005 -0.12"/> <!-- center of mass -->
-        <inertia ixx = "0.24968270"  ixy = "0.0"  ixz = "0.0"
-                 iyx = "0.0"  iyy = "0.19606323"  iyz = "0.0"
-                 izx = "0.0" izy = "0.0" izz = "0.22666109" />
-      </inertial>
+<!--      <inertial>-->
+<!--        <mass value="${mass}"/>-->
+<!--        <origin xyz="0.00056715 0.0005 -0.12"/> &lt;!&ndash; center of mass &ndash;&gt;-->
+<!--        <inertia ixx = "0.24968270"  ixy = "0.0"  ixz = "0.0"-->
+<!--                 iyx = "0.0"  iyy = "0.19606323"  iyz = "0.0"-->
+<!--                 izx = "0.0" izy = "0.0" izz = "0.22666109" />-->
+<!--      </inertial>-->
       <visual>
         <origin xyz="0 0 0" rpy="0 0 0"/>
@@ -74,6 +74,6 @@
       </plugin>
     </gazebo> -->
-    <xacro:include filename="$(find rov_description)/urdf/rov_actuators.xacro"/>
-    <xacro:include filename="$(find rov_description)/urdf/rov_sensors.xacro"/>
+<!--    <xacro:include filename="$(find rov_description)/urdf/rov_actuators.xacro"/>-->
+<!--    <xacro:include filename="$(find rov_description)/urdf/rov_sensors.xacro"/>-->
   </xacro:macro>
 </robot>

File: urdf/rov_default.xacro (robot description, xacro)
@@ -24,9 +24,23 @@
   </xacro:rov_base>
   <!-- setup base links -->
-  <link name="${namespace}/frame_link"/>
-  <joint name="${namespace}/base_frame_joint" type="fixed">
+<!--  <link name="${namespace}/frame_link"/>-->
+<!--  <joint name="${namespace}/frame_joint" type="fixed">-->
+<!--    <parent link="${namespace}/base_link"/>-->
+<!--    <child link="${namespace}/frame_link"/>-->
+<!--    <origin xyz="0 0.0373 -0.15585" rpy="0 0 0"/>-->
+<!--  </joint>-->
+  <!-- depth sensor -->
+  <link name="${namespace}/depth_sensor_link"/>
+  <joint name="${namespace}/depth_sensor_joint" type="fixed">
     <parent link="${namespace}/base_link"/>
-    <child link="${namespace}/frame_link"/>
-    <origin xyz="0 0.0373 -0.15585" rpy="0 0 0"/>
+    <child link="${namespace}/depth_sensor_link"/>
+    <origin xyz="0.1 0.1 0" rpy="${2*deg90} 0 0"/>
+  </joint>
+  <!-- Realsense T265 -->
+  <link name="t265_pose_frame"/>
+  <joint name="t265_joint" type="fixed">
+    <child link="${namespace}/base_link"/>
+    <parent link="t265_pose_frame"/>
+    <origin xyz="-0.2 0 0" rpy="0 0 ${deg90}"/>
   </joint>
   <!-- Joint state publisher plugin -->

File: urdf/rov_sensors.xacro (robot description, xacro)
@@ -108,7 +108,7 @@
   <!-- Intel Realsense Cameras -->
   <!-- RealSense D415 Camera -->
-  <xacro:include filename="$(find realsense2_description)/urdf/_d435.urdf.xacro"/>
-  <xacro:sensor_d435 parent="${namespace}/frame_link" camera_name="${namespace}/realsense_cam">
-    <origin xyz="0 0 -0.11" rpy="0 ${90*d2r} 0"/>
-  </xacro:sensor_d435>
+<!--  <xacro:include filename="$(find realsense2_description)/urdf/_d435.urdf.xacro"/>-->
+<!--  <xacro:sensor_d435 parent="${namespace}/frame_link" camera_name="${namespace}/realsense_cam">-->
+<!--    <origin xyz="0 0 -0.11" rpy="0 ${90*d2r} 0"/>-->
+<!--  </xacro:sensor_d435>-->
 </robot>
