Commit message: Working lat long pids

File: urdf/rov_default.xacro (robot description, xacro)
@@ -42,5 +42,5 @@
     <child link="${namespace}/base_link"/>
     <parent link="t265_pose_frame"/>
-    <origin xyz="-0.2 0 0" rpy="0 0 ${deg90}"/>
+    <origin xyz="-0.2 0 0.075" rpy="${-1.0*deg90/3} 0 ${deg90}"/>
   </joint>
   <!-- Joint state publisher plugin -->
